File: PCB/Weatherstation.kicad_pcb (KiCad board)
At the start: 2 copper layers, 61.5 x 59.5 mm, 11 parts, among them SW1 SW_SPDT, U1 DHT11, U2 TFT_ST7735_SD, U4 WEMOS_C3_Mini, U5 EC11B

Commit message: add case and code
Parts:
- moved SW1 54.8 mm to (123.0, 94.5)
- moved U4 1.89 mm to (133.6, 54.4)
Routing:
- net Net-(SW1-B): track 17.7 -> 85.5 mm
- net TP_input: track 20.5 -> 71.9 mm
- net (no net): track 50.9 -> 0.00 mm
- net CS: track 28.3 -> 56.7 mm
- net SCK: track 95.5 -> 74.5 mm, vias 0 -> 1
- net VCC: track 38.4 -> 59.1 mm, vias 0 -> 1
- net DATA: track 93.1 -> 75.6 mm, vias 2 -> 1
- net MOSI: track 89.1 -> 77.6 mm, vias 0 -> 1
- net ENC_C: track 62.3 -> 52.0 mm, vias 2 -> 1
- net ENC_B: track 63.4 -> 54.0 mm
- net +3V3: track 111.4 -> 102.7 mm
- net D/C: track 31.2 -> 37.7 mm, vias 0 -> 2
- net ENC_A: track 46.5 -> 41.9 mm, vias 2 -> 0
- net EN: track 5.15 -> 6.58 mm
- net MISO: track 51.2 -> 52.4 mm, vias 1 -> 0
Other:
- outline, holes or cut-outs redrawn
